File: cp_midi_control_surface_002_module_template.kicad_pcb (KiCad board)
At the start: 2 copper layers, 20 parts, among them J1 Conn_02x03_Counter_Clockwise, J10 Conn_02x18_Odd_Even, J11 Conn_02x03_Counter_Clockwise, J12 Conn_02x05_Odd_Even, J13 Conn_02x03_Counter_Clockwise, J14 Conn_02x03_Counter_Clockwise, J15 Conn_02x03_Counter_Clockwise, J16 Conn_02x03_Odd_Even, J2 Conn_02x03_Counter_Clockwise, J3 Conn_02x03_Counter_Clockwise, J4 Conn_02x03_Counter_Clockwise, J5 Conn_02x03_Counter_Clockwise, J6 Conn_02x03_Counter_Clockwise, J7 Conn_02x03_Counter_Clockwise, J8 Conn_02x03_Counter_Clockwise, J9 Conn_02x03_Counter_Clockwise, U1 CD74HC4067M, U2 CD74HC4067M, U3 CD74HC4067M, U4 CD74HC4067M

Commit message: Update cp_midi_control_surface_002_module_template.kicad_pcb
Parts:
- moved J10 54.6 mm to (153.7, 203.2)
- moved J11 54.6 mm to (189.2, 203.2)
- moved J12 54.6 mm to (245.1, 203.2)
- moved J13 54.6 mm to (301.0, 203.2)
- moved J14 54.6 mm to (356.9, 203.2)
- moved J15 54.6 mm to (412.8, 203.2)
- moved J16 54.6 mm to (468.6, 203.2)
- moved J9 54.6 mm to (97.8, 203.2)
- moved J1 54.6 mm to (97.8, 104.1)
- moved J2 54.6 mm to (153.7, 104.1)
- moved J3 54.6 mm to (189.2, 104.1)
- moved J4 54.6 mm to (245.1, 104.1)
- moved J5 54.6 mm to (301.0, 104.1)
- moved J6 54.6 mm to (356.9, 104.1)
- moved J7 54.6 mm to (412.8, 104.1)
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